Commit message: moved Ur10 to accessories

File: ridgeback/ridgeback_description/urdf/accessories.urdf.xacro (robot description, xacro)
@@ -11,5 +11,5 @@
   <xacro:include filename="$(find ridgeback_description)/urdf/accessories/sick_lms1xx_mount.urdf.xacro" />
   <xacro:include filename="$(find ridgeback_description)/urdf/accessories/hokuyo_ust-10lx_mount.urdf.xacro" />
-  <xacro:include filename="$(find ur_description)/urdf/ur5.urdf.xacro" />
+  <xacro:include filename="$(find ur_description)/urdf/ur10.urdf.xacro" />
   <xacro:include filename="$(find robotiq_s_model_visualization)/cfg/s-model_articulated_macro.xacro" />
   <!-- If enabled, generate the front HOKUYO UST-10LX LASER payload. -->
@@ -55,9 +55,9 @@
   </joint>
 <!-- Spawn arm -->
-  <xacro:ur5_robot prefix="ur5_arm_" joint_limited="true"/>
+  <xacro:ur10_robot prefix="ur10_arm_" joint_limited="true"/>
   <!-- Join arm -->
-  <joint name="ur5_arm_base" type="fixed">
+  <joint name="ur10_arm_base" type="fixed">
 	<parent link="arch_link" />
-	<child link="ur5_arm_base_link" />
+	<child link="ur10_arm_base_link" />
 	<origin xyz="0.01 -0.27 0.375" rpy="0.0 0.0 1.571" />
   </joint>
@@ -65,5 +65,5 @@
   <xacro:s-model_articulated prefix="" />
   <joint name="gripper_base" type="fixed">
-	<parent link="ur5_arm_ee_link" />
+	<parent link="ur10_arm_ee_link" />
 	<child link="palm" />
 	<origin xyz="0.11 0.0 0.0" rpy="0.0 -0.786 -1.57" />
@@ -85,5 +85,5 @@
   <joint name="FT300_joint" type="fixed">
 	  <origin xyz="0.03 0 0" rpy="0 1.57 0" />
-	  <parent link="ur5_arm_ee_link" />
+	  <parent link="ur10_arm_ee_link" />
 	  <child link="FT300_link" />
   </joint>

File: ridgeback/ridgeback_description/urdf/ridgeback.urdf.xacro (robot description, xacro)
@@ -198,38 +198,4 @@
     <origin xyz="0 0 ${deck_height}" rpy="0 0 0"/>
   </joint>
-  <!-- Spawn arm -->
-  <xacro:ur10_robot prefix="ur10_arm_" joint_limited="true"/>
-  <!-- Join arm -->
-  <joint name="ur10_arm_base" type="fixed">
-    <parent link="top_link" />
-    <child link="ur10_arm_base_link" />
-    <origin xyz="0.3058 0 0.0065" rpy="0.0 0.0 -1.57" />
-  </joint>
-  <!-- Spawn and Join Gripper -->
-  <xacro:s-model_articulated prefix="" />
-  <joint name="gripper_base" type="fixed">
-    <parent link="ur10_arm_ee_link" />
-      <child link="palm" />
-      <origin xyz="0.11 0.0 0.0" rpy="0.0 -0.784 -1.57" />
-  </joint>
-  <!-- Sensor Mount and other custom parts -->
-  <link name="FT300_link">
-    <visual>
-      <geometry>
-        <cylinder length="0.06" radius="0.035"/>
-      </geometry>
-      <material name="black"/>
-    </visual>
-	<collision>
-		<geometry>
-			<cylinder length="0.055" radius="0.035"/>
-		</geometry>
-	</collision>
-  </link>
-  <joint name="FT300_joint" type="fixed">
-	  <origin xyz="0.03 0 0" rpy="0 1.57 0" />
-	  <parent link="ur10_arm_ee_link" />
-	  <child link="FT300_link" />
-  </joint>
   <!-- Bring in simulation data for Gazebo. -->
   <xacro:include filename="$(find ridgeback_description)/urdf/ridgeback.gazebo" />

Commit message: tuned arm rotation, good to plan now

File: ridgeback/ridgeback_description/urdf/accessories.urdf.xacro (robot description, xacro)
@@ -60,5 +60,5 @@
 	<parent link="arch_link" />
 	<child link="ur10_arm_base_link" />
-	<origin xyz="0.01 -0.27 0.375" rpy="0.0 0.0 1.571" />
+	<origin xyz="0.01 -0.27 0.375" rpy="0.0 0.0 3.1416" />
   </joint>
   <!-- Spawn and Join Gripper -->
